File: Kicad/a0/a0.kicad_sch (KiCad schematic)
At the start: 73 parts, among them J1 Conn_02x03_Odd_Even, J2 VGA, J4 AudioJack3_SwitchTR, J5 Conn_02x17_Odd_Even, J6 Barrel_Jack_MountingPin, J7 DE9_Plug, J8 DE9_Plug, SW1 SW_Push_45deg, SW10 SW_Push_45deg, SW11 SW_Push_45deg, SW12 SW_Push_45deg, SW13 SW_Push_45deg, SW14 SW_Push_45deg, SW15 SW_Push_45deg, SW16 SW_Push_45deg, SW17 SW_Push_45deg, SW18 SW_Push_45deg, SW19 SW_Push_45deg, SW2 SW_Push_45deg, SW20 SW_Push_45deg, SW21 SW_Push_45deg, SW22 SW_Push_45deg, SW23 SW_Push_45deg, SW24 SW_Push_45deg, SW25 SW_Push_45deg, SW26 SW_Push_45deg, SW27 SW_Push_45deg, SW28 SW_Push_45deg, SW29 SW_Push_45deg, SW3 SW_Push_45deg, SW30 SW_Push_45deg, SW31 SW_Push, SW32 SW_SPDT, SW4 SW_Push_45deg, SW5 SW_Push_45deg, SW6 SW_Push_45deg, SW7 SW_Push_45deg, SW8 SW_Push_45deg, SW9 SW_Push_45deg, U1 74HC590A, U10 74LS541, U11 74LS166, U2 74HC590A, U3 74LS14, U4 74LS174, U5 4520, U6 74LS32, U7 74LS10, U8 CY62256-70PC, U9 28C256, Y1 Crystal

Commit message: pcb,bios,font  improvements
Parts:
- removed J4: AudioJack3_SwitchTR, Connector_Audio:Jack_3.5mm_CUI_SJ1-3525N_Horizontal, symbol Connector_Audio:AudioJack3_SwitchTR
- removed U9: 28C256, Package_DIP:DIP-28_W15.24mm_LongPads, symbol Memory_EEPROM:28C256
- added C16: 10µF, PCM_Capacitor_THT_AKL:CP_Radial_D5.0mm_P2.00mm, symbol Device:C_Polarized
- added C3: 4.7µF, PCM_Capacitor_THT_AKL:CP_Radial_D5.0mm_P2.00mm, symbol PCM_Capacitor_AKL:CP_Radial_D5.0mm_P2.00mm
- added D10, D11, D12, D13, D14, D15, D16, D17, D18, D19, D2, D20, D21, D22, D23, D24, D25, D26, D27, D28, D29, D3, D30, D31, D32, D33, D34, D35, D36, D37, D38, D4, D5, D6, D7, D8, D9: 1N4148, PCM_Diode_THT_AKL:D_DO-35_SOD27_P7.62mm_Horizontal, symbol PCM_Diode_AKL:1N4148
- added H1, H2: MountingHole, MountingHole:MountingHole_2.2mm_M2, symbol Mechanical:MountingHole
- added J3: AudioJack4, Connector_Audio:Jack_3.5mm_PJ320E_Horizontal, symbol Connector_Audio:AudioJack4
- added R10, R15, R9: 3.3kΩ, PCM_Resistor_THT_AKL:R_Axial_DIN0204_L3.6mm_D1.6mm_P5.08mm_Horizontal, symbol Device:R
- added R11: 5.6KΩ, PCM_Resistor_THT_US_AKL:R_Axial_DIN0204_L3.6mm_D1.6mm_P1.90mm_Vertical, symbol Device:R
- added R12, R13: 27KΩ, PCM_Resistor_THT_US_AKL:R_Axial_DIN0204_L3.6mm_D1.6mm_P1.90mm_Vertical, symbol Device:R
- added R14: 20KΩ, PCM_Resistor_THT_AKL:R_Axial_DIN0204_L3.6mm_D1.6mm_P5.08mm_Horizontal, symbol Device:R
- added R6, R7, R8: R_Small, PCM_Resistor_THT_AKL:R_Axial_DIN0204_L3.6mm_D1.6mm_P1.90mm_Vertical, symbol Device:R_Small
- added RN1: R_Network06, Resistor_THT:R_Array_SIP7, symbol Device:R_Network06
- added U4: SST39SF040, Package_DIP:DIP-32_W15.24mm_LongPads, symbol Memory_Flash:SST39SF040
- BZ1: footprint Buzzer_Beeper:MagneticBuzzer_Kobitone_254-EMB73-RO -> Connector_PinHeader_2.54mm:PinHeader_1x02_P2.54mm_Vertical
- J6: value Barrel_Jack_MountingPin -> Barrel Jack
- R1: value R -> 1MΩ; footprint PCM_Resistor_THT_US_AKL_Double:R_Axial_DIN0204_L3.6mm_D1.6mm_P5.08mm_Horizontal -> PCM_Resistor_THT_AKL:R_Axial_DIN0204_L3.6mm_D1.6mm_P5.08mm_Horizontal
- R2: value R -> 10KΩ; footprint PCM_Resistor_THT_US_AKL_Double:R_Axial_DIN0204_L3.6mm_D1.6mm_P5.08mm_Horizontal -> PCM_Resistor_THT_AKL:R_Axial_DIN0204_L3.6mm_D1.6mm_P5.08mm_Horizontal
- R4: value R -> 330Ω; footprint PCM_Resistor_THT_US_AKL_Double:R_Axial_DIN0204_L3.6mm_D1.6mm_P5.08mm_Horizontal -> PCM_Resistor_THT_AKL:R_Axial_DIN0204_L3.6mm_D1.6mm_P5.08mm_Horizontal
- R5: value R -> 100Ω; footprint PCM_Resistor_THT_US_AKL_Double:R_Axial_DIN0204_L3.6mm_D1.6mm_P5.08mm_Horizontal -> PCM_Resistor_THT_AKL:R_Axial_DIN0204_L3.6mm_D1.6mm_P5.08mm_Horizontal
- SW1: value SW_Push_45deg -> Q
- SW10: value SW_Push_45deg -> P
- SW11: value SW_Push_45deg -> A
- SW12: value SW_Push_45deg -> S
- SW13: value SW_Push_45deg -> D
- SW14: value SW_Push_45deg -> F
- SW15: value SW_Push_45deg -> G
- SW16: value SW_Push_45deg -> H
- SW17: value SW_Push_45deg -> J
- SW18: value SW_Push_45deg -> K
- SW19: value SW_Push_45deg -> L
- SW2: value SW_Push_45deg -> W
- SW20: value SW_Push_45deg -> ENTER
- SW21: value SW_Push_45deg -> Z
- SW22: value SW_Push_45deg -> X
- SW23: value SW_Push_45deg -> C
- SW24: value SW_Push_45deg -> V
- SW25: value SW_Push_45deg -> SHIFT
- SW26: value SW_Push_45deg -> ALT
- SW27: value SW_Push_45deg -> B
- SW28: value SW_Push_45deg -> N
- SW29: value SW_Push_45deg -> M
- SW3: value SW_Push_45deg -> E
- SW30: value SW_Push_45deg -> SPACE
- SW4: value SW_Push_45deg -> R
- SW5: value SW_Push_45deg -> T
- SW6: value SW_Push_45deg -> Y
- SW7: value SW_Push_45deg -> U
- SW8: value SW_Push_45deg -> I
- SW9: value SW_Push_45deg -> O
- U10: renamed from U6; value 74LS32 -> 74HC32
- U11: renamed from U4; value 74LS174 -> 74HC174
- U12: renamed from U5; value 4520 -> 74HC4520
- U5: renamed from U12; value ~ -> 65C02
- U6: renamed from U10; value 74LS541 -> 74HCT541
- U7: renamed from U11; value 74LS166 -> 74HC166
- U8: renamed from U3; value 74LS14 -> 74HC14
- U9: renamed from U7; value 74LS10 -> 74HC10
- Y1: value Crystal -> 32Mhz
- renumbered U2 to U1, U1 to U2, U8 to U3
Connections:
- net A0: now also J5.11 (Pin_11), U9.11, D2.1 (K), U4.12 (A0); no longer U11.11 (D3)
- net A1: now also J5.13 (Pin_13), U9.10, D3.1 (K), U4.11 (A1); no longer U11.6 (D2)
- net A10: now also J5.31 (Pin_31), U4.23 (A10)
- net A11: now also J5.33 (Pin_33), U4.25 (A11)
- net A12: now also J5.32 (Pin_32), D37.1 (K), U4.4 (A12)
- net A13: now also J5.30 (Pin_30), D38.1 (K), R8.2, U4.28 (A13)
- net A14: now also J5.28 (Pin_28), R7.2, U4.29 (A14)
- net A15: now also J5.26 (Pin_26), R6.2
- net A2: now also J5.15 (Pin_15), U9.4, D4.1 (K), U4.10 (A2); no longer U11.4 (D1)
- net A3: now also J5.17 (Pin_17), D5.1 (K), U4.9 (A3)
- net A4: now also J5.19 (Pin_19), D6.1 (K), U4.8 (A4)
- net A5: now also J5.21 (Pin_21), U4.7 (A5)
- net A6: now also J5.23 (Pin_23), U4.6 (A6)
- net A7: now also J5.25 (Pin_25), U4.5 (A7)
- net A8: now also J5.27 (Pin_27), U4.27 (A8)
- net A9: now also J5.29 (Pin_29), U4.26 (A9)
- net AUDIN: now also J3.S
- net BEEP: now also R14.1
- net D0: now also J5.10 (Pin_10), U4.13 (D0)
- net D1: now also J5.12 (Pin_12), U4.14 (D1)
- net D2: now also J5.14 (Pin_14), U4.15 (D2)
- net D3: now also J5.16 (Pin_16), U4.17 (D3)
- net D4: now also J5.18 (Pin_18), U4.18 (D4)
- net D5: now also J5.20 (Pin_20), U4.19 (D5)
- net D6: now also J5.22 (Pin_22), U4.20 (D6)
- net D7: now also J5.24 (Pin_24), U4.21 (D7)
- net GND: now also C10.1, C11.1, C12.1, C13.1, C14.1, C15.1, C4.1, C5.1, C6.1, C7.1, C8.1, J5.1 (Pin_1), J5.34 (Pin_34), U10.7 (GND), U11.8 (GND), U12.8 (VSS), U3.14 (GND), U5.21 (VSS), U6.10 (GND), U8.7 (GND), U9.7 (GND), C16.2, J3.R1, R13.1, R6.1, R7.1, R8.1, U4.16 (GND)
- net H32: now also U11.13 (D4)
- net H32': now also U11.12 (Q4)
- net RAMDIS: now also J5.9 (Pin_9)
- net ROMDIS: now also J5.7 (Pin_7), U4.22 (CE)
- net V1: now also U9.5; no longer U11.13 (D4)
- net V512: now also U11.4 (D1), U9.3, U9.9; no longer U11.3 (D0)
- net V512': now also U11.5 (Q1); no longer U11.2 (Q0), U9.3, U9.9
- net VCC: now also J5.2 (Pin_2), SW31.2, U5.38 (~{SO}), C16.1, C3.1, R10.1, R15.1, R9.1, RN1.1 (common), U4.1 (A18), U4.2 (A16), U4.3 (A15), U4.30 (A17), U4.31 (PGM), U4.32 (VCC)
- net r/~{w}: now also U5.34 (R/~{W}), R10.2
- net ~{MRC}: now also U11.7 (Q2); no longer U9.6
- net ~{UPPER}: now also U4.24 (OE)
- net ~{VSYNC}: now also J5.3 (Pin_3), U11.10 (Q3), U5.4 (~{IRQ}); no longer U9.8
- net ~{WR}: now also J5.8 (Pin_8)
- net ø2: now also J5.4 (Pin_4), U5.36 (BE), U5.37 (ø0)
- net COL 2: now reaches SW26.1
- net COL 2: now also SW15.1, SW16.1, SW25.1, SW5.1, SW6.1, D4.2 (A)
- net at SW26.2: now also D34.1 (K)
- net at SW32.1 (A): now also J6.1
- net at SW32.3 (C): no longer J6.1
- net HROW 0: now reaches J8.1
- net HROW 0: now also J7.1, U6.2 (A0), D10.2 (A), D11.2 (A), D7.2 (A), D8.2 (A), D9.2 (A), RN1.2 (R1)
- net HROW 1: now reaches J8.2
- net HROW 1: now also J7.2, U6.3 (A1), D17.2 (A), D18.2 (A), D19.2 (A), D20.2 (A), D21.2 (A), RN1.3 (R2)
- net HROW 2: now reaches J8.3
- net HROW 2: now also J7.3, U6.4 (A2), D27.2 (A), D28.2 (A), D29.2 (A), D30.2 (A), D31.2 (A), RN1.4 (R3)
- net HROW 3: now reaches J8.4
- net HROW 3: now also J7.4, U6.5 (A3), D32.2 (A), D33.2 (A), D34.2 (A), D35.2 (A), D36.2 (A), RN1.5 (R4)
- net HROW 4: now reaches J8.6
- net HROW 4: now also J7.6, U6.6 (A4), D22.2 (A), D23.2 (A), D24.2 (A), D25.2 (A), D26.2 (A), RN1.6 (R5)
- net at J8.8: now also D37.2 (A)
- net HROW 5: now reaches J8.9
- net HROW 5: now also J7.9, U6.7 (A5), D12.2 (A), D13.2 (A), D14.2 (A), D15.2 (A), D16.2 (A), RN1.7 (R6)
- net COL 0: now reaches SW2.1
- net COL 0: now also SW1.1, SW11.1, SW12.1, SW21.1, SW22.1, D2.2 (A)
- net at SW2.2: now also D16.1 (K)
- net at SW1.2: now also D7.1 (K)
- net at U5.2 (RDY): now also R9.2
- net ~{RESEŦ}: now reaches U5.40 (~{RESET})
- net ~{RESEŦ}: now also J5.5 (Pin_5), U8.12
- net ~{NMI}: now reaches U5.6 (~{NMI})
- net ~{NMI}: now also J5.6 (Pin_6), R15.2
- net COL 4: now reaches SW30.1
- net COL 4: now also SW10.1, SW19.1, SW20.1, SW29.1, SW9.1, D6.2 (A)
- net at SW30.2: now also D36.1 (K)
- net COL 3: now reaches SW27.1
- net COL 3: now also SW17.1, SW18.1, SW28.1, SW7.1, SW8.1, D5.2 (A)
- net at SW27.2: now also D30.1 (K)
- net at SW6.2: now also D14.1 (K)
- net COL 1: now reaches SW3.1
- net COL 1: now also SW13.1, SW14.1, SW23.1, SW24.1, SW4.1, D3.2 (A)
- net at SW3.2: now also D8.1 (K)
- net at SW20.2: now also D26.1 (K)
- net at SW16.2: now also D24.1 (K)
- net at SW29.2: now also D31.1 (K)
- net at SW28.2: now also D35.1 (K)
- net at J7.8: now also D38.2 (A)
- net at SW31.1: now also R12.1, R13.2
- net at U8.13: now also R11.2
- net at SW22.2: now also D32.1 (K)
- net at SW12.2: now also D22.1 (K)
- net at SW18.2: now also D25.1 (K)
- net at SW8.2: now also D13.1 (K)
- net at SW23.2: now also D28.1 (K)
- net at SW4.2: now also D15.1 (K)
- net at SW9.2: now also D11.1 (K)
- net at SW7.2: now also D10.1 (K)
- net at SW10.2: now also D12.1 (K)
- net at SW21.2: now also D27.1 (K)
- net at SW17.2: now also D20.1 (K)
- net at SW5.2: now also D9.1 (K)
- net at SW14.2: now also D23.1 (K)
- net at SW15.2: now also D19.1 (K)
- net at SW24.2: now also D33.1 (K)
- net at SW11.2: now also D17.1 (K)
- net at SW13.2: now also D18.1 (K)
- net at SW25.2: now also D29.1 (K)
- net at SW19.2: now also D21.1 (K)
- removed net V1': U11.12 (Q4), U9.5
- removed net V2': U11.10 (Q3), U9.11
- removed net V4': U11.7 (Q2), U9.10
- removed net V8': U11.5 (Q1), U9.4
- new net: U11.11 (D3), U9.8
- new net: U11.6 (D2), U9.6
- new net: C3.2, R11.1, R12.2
- new net: J3.T, R14.2
- no-connect marks 8 -> 20
Other:
- moved on the sheet: BZ1, C10, C11, C12, C13, C14, C15, C4, C5, C6, C7, C8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

Commit message: update system logic
Parts:
- removed R6, R7, R8: R_Small, PCM_Resistor_THT_AKL:R_Axial_DIN0204_L3.6mm_D1.6mm_P1.90mm_Vertical, symbol Device:R_Small
- removed RN1: R_Network06, Resistor_THT:R_Array_SIP7, symbol Device:R_Network06
- removed U5: 65C02, Package_DIP:DIP-40_W15.24mm_LongPads, symbol MM:65c02
- added R16: 3.3kΩ, PCM_Resistor_THT_AKL:R_Axial_DIN0204_L3.6mm_D1.6mm_P5.08mm_Horizontal, symbol Device:R
- added R18: R_Small, PCM_Resistor_THT_AKL:R_Axial_DIN0204_L3.6mm_D1.6mm_P1.90mm_Vertical, symbol Device:R_Small
- added RN1, RN2: R_Network08, Resistor_THT:R_Array_SIP9, symbol Device:R_Network08
- added U5: W65C02SxP, Package_DIP:DIP-40_W15.24mm, symbol PCM_65xx-library:W65C02SxP
- C1, C2: value C_Small -> 33pF
Connections:
- net V1 is gone; now on net A1: U2.6 (Q6), U9.5
- net A0: now also U5.9 (A0)
- net A1: now also U5.10 (A1); no longer U9.10
- net A10: now also U5.19 (A10)
- net A11: now also U5.20 (A11)
- net A12: now also J5.34 (Pin_34), U5.22 (A12); no longer J5.32 (Pin_32)
- net A13: now also J5.32 (Pin_32), U8.5, RN2.2 (R1), U5.23 (A13); no longer J5.30 (Pin_30)
- net A14: now also J5.30 (Pin_30), RN2.3 (R2), U5.24 (A14); no longer J5.28 (Pin_28), U8.5
- net A15: now also J5.28 (Pin_28), RN2.4 (R3), U5.25 (A15); no longer J5.26 (Pin_26)
- net A2: now also U9.10, U5.11 (A2)
- net A3: now also U5.12 (A3)
- net A4: now also U5.13 (A4)
- net A5: now also U5.14 (A5)
- net A6: now also U5.15 (A6)
- net A7: now also U10.10, U5.16 (A7); no longer U8.11
- net A8: now also U5.17 (A8)
- net A9: now also U5.18 (A9)
- net D0: now also U5.33 (D0)
- net D1: now also U5.32 (D1)
- net D2: now also U5.31 (D2)
- net D3: now also U5.30 (D3)
- net D4: now also U5.29 (D4)
- net D5: now also U5.28 (D5)
- net D6: now also U5.27 (D6)
- net D7: now also U5.26 (D7)
- net GND: now also R18.1, RN2.1 (common), U5.21 (VSS); no longer J5.34 (Pin_34)
- net H32: now also U10.1, U8.11; no longer U10.10
- net H32': now also U10.2; no longer U7.9 (Clr)
- net HROW 0: now also RN1.2 (R1)
- net HROW 1: now also RN1.3 (R2)
- net HROW 2: now also RN1.4 (R3)
- net HROW 3: now also RN1.5 (R4)
- net HROW 4: now also RN1.6 (R5)
- net HROW 5: now also RN1.7 (R6)
- net RAMDIS: now also R18.2, RN2.5 (R4)
- net ROMDIS: now also RN2.6 (R5); no longer J5.7 (Pin_7), U4.22 (CE)
- net VCC: now also R10.2, R16.1, RN1.1 (common), U5.8 (VDD); no longer R10.1
- net r/~{w}: now also R10.1, U5.34 (R/~{W}); no longer R10.2
- net ~{NMI}: now also U5.6 (~{NMI})
- net ~{RESEŦ}: now also U5.40 (~{RES}); no longer J5.5 (Pin_5)
- net ~{VSYNC}: now also U5.4 (~{IRQ})
- net ø2: now also U5.36 (BE), U5.37 (ϕ0)
- net ~{A13}: now reaches U8.6
- net ~{A13}: now also U4.22 (CE); no longer U10.1
- net at R9.2: now also U5.2 (RDY)
- net ~{A15}: now reaches U6.1 (G1), U8.2
- net ~{A15}: now also U4.24 (OE); no longer U10.2
- net ~{UPPER}: no longer names the net of U10.3
- net ~{UPPER}: now also U7.9 (Clr); no longer U4.24 (OE)
- new net: R16.2, U5.38 (~{SO})
- new net DataOut: RN2.8 (R7)
- new net NMI: RN1.9 (R8)
- new net R/W: RN1.8 (R7)
- new net Speaker: RN2.7 (R6)
- new net ~{RESET}: J5.5 (Pin_5)
- no-connect marks 20 -> 21
Other:
- note added: "16K ROM"
- note added: "32K RAM"
- note added: "522-523"
- note added: "=524"
- note added: "CPU"
- note added: "Clock"
- note added: "Expansion Slot"
- note added: "Keyboard and Joysticks"
- note added: "Pixel Shifter"
- note added: "Power Input"
- note added: "Reset"
- note added: "Video Counters"
- note added: "Video Signal Buffer"
- note removed: "518-519"
- note removed: "=521"
- moved on the sheet: BZ1, C10, C12, C13, C14, C15, C16, C3, C4, C5, C6, C7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

Commit message: file update
Parts:
- removed R10, R15, R16: 3.3kΩ, PCM_Resistor_THT_AKL:R_Axial_DIN0204_L3.6mm_D1.6mm_P5.08mm_Horizontal, symbol Device:R
- R14, R5: footprint PCM_Resistor_THT_AKL:R_Axial_DIN0204_L3.6mm_D1.6mm_P5.08mm_Horizontal -> PCM_Resistor_THT_US_AKL:R_Axial_DIN0204_L3.6mm_D1.6mm_P1.90mm_Vertical
- R3: footprint Resistor_THT:R_Axial_DIN0204_L3.6mm_D1.6mm_P5.08mm_Horizontal -> PCM_Resistor_THT_AKL:R_Axial_DIN0204_L3.6mm_D1.6mm_P5.08mm_Horizontal
Connections:
- net ROMDIS is gone; now on net A14: RN2.6 (R5)
- net R/W is gone; now on net HROW 4: RN1.8 (R7)
- net A1: now also U9.13; no longer U9.5
- net A11: now also D37.1 (K)
- net A12: now also D38.1 (K); no longer D37.1 (K)
- net A13: now also RN2.5 (R4); no longer D38.1 (K), RN2.2 (R1)
- net A14: no longer RN2.3 (R2)
- net A15: now also RN2.7 (R6); no longer RN2.4 (R3)
- net A2: now also U9.2; no longer U9.4
- net A6: now also U8.3; no longer U10.9
- net A7: now also U10.9; no longer U10.10
- net BEEP: now also R5.1; no longer BZ1.1 (+)
- net D0: now also J5.12 (Pin_12); no longer J5.10 (Pin_10)
- net D1: now also J5.14 (Pin_14); no longer J5.12 (Pin_12)
- net D2: now also J5.16 (Pin_16); no longer J5.14 (Pin_14)
- net D3: now also J5.18 (Pin_18); no longer J5.16 (Pin_16)
- net D4: now also J5.20 (Pin_20); no longer J5.18 (Pin_18)
- net D5: now also J5.22 (Pin_22); no longer J5.20 (Pin_20)
- net D6: now also J5.24 (Pin_24); no longer J5.22 (Pin_22)
- net D7: now also J5.26 (Pin_26); no longer J5.24 (Pin_24)
- net DataOut: now also J3.T, R14.2, RN2.4 (R3); no longer RN2.8 (R7)
- net GND: now also BZ1.2 (-); no longer R5.2
- net H32: now also U10.10; no longer U8.11
- net HROW 0: now also RN1.4 (R3); no longer RN1.2 (R1)
- net HROW 1: now also RN1.5 (R4); no longer RN1.3 (R2)
- net HROW 2: now also RN1.6 (R5); no longer RN1.4 (R3)
- net HROW 3: now also RN1.7 (R6); no longer RN1.5 (R4)
- net HROW 4: no longer RN1.6 (R5)
- net HROW 5: now also RN1.9 (R8); no longer RN1.7 (R6)
- net M16: now also J5.3 (Pin_3)
- net M2: now also U9.5; no longer U9.13
- net M4: now also U9.4; no longer U9.2
- net M8: now also U9.3; no longer U9.1
- net NMI: now also RN1.3 (R2); no longer RN1.9 (R8)
- net Speaker: now also BZ1.1 (+), R5.2, RN2.3 (R2); no longer RN2.7 (R6)
- net V512: now also U9.1; no longer U9.3
- net VCC: now also U5.38 (~{SO})
- net r/~{w}: now also J5.10 (Pin_10), RN1.2 (R1)
- net ~{A13}: now also J5.9 (Pin_9)
- net ~{A15}: now also J5.8 (Pin_8)
- net ~{RESET}: now also U5.40 (~{RES}), U8.10
- net ~{VSYNC}: no longer J5.3 (Pin_3)
- net ~{WR}: no longer J5.8 (Pin_8)
- net ~{sload}: now also U9.6; no longer U9.12
- net ø1: now also U8.13; no longer U8.3
- net ø2: now also U8.12; no longer U8.4
- net at U11.6 (D2): now also U9.12; no longer U9.6
- net at U10.12: now also U8.4; no longer U10.8
- net at U10.13: now also U10.8; no longer U8.10
- net at R11.2: now also U8.11; no longer U8.13
- net RAMHIDE: now reaches J5.7 (Pin_7)
- net RAMHIDE: now also R18.2, U3.22 (~{OE})
- removed net RAMDIS: J5.9 (Pin_9), R18.2, RN2.5 (R4), U3.22 (~{OE})
- removed net ~{RESEŦ}: U5.40 (~{RES}), U8.12
- no-connect marks 21 -> 23
Other:
- note added: "Keyboard"
- note removed: "Keyboard and Joysticks"
- moved on the sheet: BZ1, J5, J7, J8, RN1, RN2, U10C, U8B, U8F, U9A, U9B
