File: Kicad/a1/a1.kicad_sch (KiCad schematic)
At the start: 126 parts, among them J1 Conn_02x03_Odd_Even, J2 VGA, J3 AudioJack4, J4 Conn_02x17_Odd_Even, J6 Barrel Jack, J7 DE9_Plug, J8 DE9_Plug, SW1 Q, SW10 P, SW11 A, SW12 S, SW13 D, SW14 F, SW15 G, SW16 H, SW17 J, SW18 K, SW19 L, SW2 W, SW20 ENT, SW21 SHIFT, SW22 Z, SW23 X, SW24 C, SW25 V, SW26 B, SW27 N, SW28 M, SW29 SPACE, SW3 E, SW30 ALT, SW31 SW_Push, SW32 SW_SPDT, SW4 R, SW5 T, SW6 Y, SW7 U, SW8 I, SW9 O, U1 74HC590A, U10 74HC32, U11 74HC174, U12 74HC4520, U2 74HC590A, U3 62256, U4 SST39SF0x0, U5 W65C02SxP, U6 74HCT540, U7 74HC166, U8 74HC14, U9 74HC10, Y1 16Mhz

Commit message: tweak clock circuit
Connections:
- net M16: now also U12.3 (Q1); no longer C2.1, R2.2, U12.2 (Enable), U8.8, Y1.2
- net M2: now also U12.6 (Q4); no longer U12.5 (Q3)
- net M4: now also U12.5 (Q3); no longer U12.4 (Q2)
- net M8: now also U12.4 (Q2); no longer U12.3 (Q1)
- new net: C2.1, R2.2, U12.2 (Enable), U8.8, Y1.2
- no-connect marks 17 -> 16
Changed lines of the file:
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@@
 	)
 	(junction
+		(at 99.06 88.9)
+		(diameter 0)
+		(color 0 0 0 0)
+	)
+	(junction
 		(at 280.67 39.37)
 		(diameter 0)
@@
 	)
 	(no_connect
-		(at 82.55 91.44)
-	)
-	(no_connect
 		(at 60.96 125.73)
 	)
@@
 		)
 	)
+	(wire
+		(pts
+			(xy 99.06 91.44) (xy 99.06 88.9)
+		)
+		(stroke
+			(width 0)
+			(type default)
+		)
+	)
 	(bus
 		(pts
@@
 		)
 	)
+	(wire
+		(pts
+			(xy 82.55 86.36) (xy 86.36 86.36)
+		)
+		(stroke
+			(width 0)
+			(type default)
+		)
+	)
 	(bus
 		(pts
@@
 		)
 	)
-	(wire
+	(bus
 		(pts
-			(xy 82.55 83.82) (xy 86.36 83.82)
+			(xy 212.09 69.85) (xy 212.09 116.84)
 		)
 		(stroke
@@
 		)
 	)
-	(bus
+	(wire
 		(pts
-			(xy 212.09 69.85) (xy 212.09 116.84)
+			(xy 262.89 67.31) (xy 267.97 67.31)
 		)
 		(stroke
@@
 	(wire
 		(pts
-			(xy 262.89 67.31) (xy 267.97 67.31)
+			(xy 57.15 226.06) (xy 57.15 254)
 		)
 		(stroke
@@
 	(wire
 		(pts
-			(xy 57.15 226.06) (xy 57.15 254)
+			(xy 303.53 160.02) (xy 303.53 165.1)
 		)
 		(stroke
@@
 	(wire
 		(pts
-			(xy 303.53 160.02) (xy 303.53 165.1)
+			(xy 82.55 88.9) (xy 86.36 88.9)
 		)
 		(stroke
@@
 	(wire
 		(pts
+			(xy 82.55 91.44) (xy 86.36 91.44)
+		)
+		(stroke
+			(width 0)
+			(type default)
+		)
+	)
+	(wire
+		(pts
 			(xy 34.29 95.25) (xy 30.48 95.25)
 		)
@@
 	(wire
 		(pts
-			(xy 82.55 88.9) (xy 86.36 88.9)
-		)
-		(stroke
-			(width 0)
-			(type default)
-		)
-	)
-	(wire
-		(pts
 			(xy 387.35 90.17) (xy 381 90.17)
 		)
@@
 	(wire
 		(pts
-			(xy 82.55 86.36) (xy 86.36 86.36)
-		)
-		(stroke
-			(width 0)
-			(type default)
-		)
-	)
-	(wire
-		(pts
 			(xy 73.66 226.06) (xy 73.66 254)
 		)
@@
 	(wire
 		(pts
-			(xy 99.06 86.36) (xy 99.06 83.82)
-		)
-		(stroke
-			(width 0)
-			(type default)
-		)
-	)
-	(wire
-		(pts
 			(xy 30.48 77.47) (xy 30.48 86.36)
 		)
@@
 		)
 	)
+	(label "M16"
+		(at 82.55 83.82 0)
+		(fields_autoplaced yes)
+		(effects
+			(font
+				(size 1.27 1.27)
+			)
+			(justify left bottom)
+		)
+	)
 	(label "A9"
 		(at 173.99 72.39 0)
@@
 		)
 	)
-	(label "M16"
-		(at 49.53 91.44 0)
-		(fields_autoplaced yes)
-		(effects
-			(font
-				(size 1.27 1.27)
-			)
-			(justify left bottom)
-		)
-	)
 	(label "HROW 2"
 		(at 151.13 218.44 90)
@@
 		)
 	)
+	(label "M4"
+		(at 82.55 88.9 0)
+		(fields_autoplaced yes)
+		(effects
+			(font
+				(size 1.27 1.27)
+			)
+			(justify left bottom)
+		)
+	)
 	(label "A6"
 		(at 173.99 64.77 0)
@@
 		)
 	)
-	(label "M2"
-		(at 82.55 88.9 0)
-		(fields_autoplaced yes)
-		(effects
-			(font
-				(size 1.27 1.27)
-			)
-			(justify left bottom)
-		)
-	)
 	(label "A1"
 		(at 168.91 52.07 180)
@@
 		)
 	)
-	(label "A7"
-		(at 168.91 67.31 180)
+	(label "M2"
+		(at 82.55 91.44 0)
 		(fields_autoplaced yes)
 		(effects
@@
 				(size 1.27 1.27)
 			)
-			(justify right bottom)
+			(justify left bottom)
 		)
 	)
-	(label "ø2"
-		(at 116.84 86.36 0)
+	(label "A7"
+		(at 168.91 67.31 180)
 		(fields_autoplaced yes)
 		(effects
@@
 				(size 1.27 1.27)
 			)
-			(justify left bottom)
+			(justify right bottom)
 		)
 	)
 	(label "ø2"
-		(at 339.09 113.03 0)
+		(at 116.84 86.36 0)
 		(fields_autoplaced yes)
 		(effects
@@
 		)
 	)
-	(label "M4"
-		(at 82.55 86.36 0)
+	(label "ø2"
+		(at 339.09 113.03 0)
 		(fields_autoplaced yes)
 		(effects
@@
 		)
 	)
-	(label "M8"
-		(at 82.55 83.82 0)
-		(fields_autoplaced yes)
-		(effects
-			(font
-				(size 1.27 1.27)
-			)
-			(justify left bottom)
-		)
-	)
 	(label "AUDIN"
 		(at 139.7 154.94 180)
@@
 		)
 	)
+	(label "M8"
+		(at 82.55 86.36 0)
+		(fields_autoplaced yes)
+		(effects
+			(font
+				(size 1.27 1.27)
+			)
+			(justify left bottom)
+		)
+	)
 	(label "H8"
 		(at 318.77 57.15 180)
@@
 	)
 	(label "ø1"
-		(at 99.06 86.36 0)
+		(at 99.06 91.44 0)
 		(fields_autoplaced yes)
 		(effects
@@
 	)
 	(symbol
+		(lib_id "Connector_Generic:Conn_02x03_Odd_Even")
+		(at 91.44 88.9 0)
+		(unit 1)
+		(exclude_from_sim no)
+		(in_bom yes)
+		(on_board yes)
+		(dnp no)
+		(property "Reference" "J1"
+			(at 92.71 83.312 0)
+			(effects
+				(font
+					(size 1.27 1.27)
+				)
+			)
+		)
+		(property "Value" "Conn_02x03_Odd_Even"
+			(at 93.218 75.946 0)
+			(effects
+				(font
+					(size 1.27 1.27)
+				)
+				(hide yes)
+			)
+		)
+		(property "Footprint" "Connector_PinHeader_2.54mm:PinHeader_2x03_P2.54mm_Vertical"
+			(at 91.44 88.9 0)
+			(effects
+				(font
+					(size 1.27 1.27)
+				)
+				(hide yes)
+			)
+		)
+		(property "Datasheet" "~"
+			(at 91.44 88.9 0)
+			(effects
+				(font
+					(size 1.27 1.27)
+				)
+				(hide yes)
+			)
+		)
+		(property "Description" "Generic connector, double row, 02x03, odd/even pin numbering scheme (row 1 odd numbers, row 2 even numbers), script generated (kicad-library-utils/schlib/autogen/connector/)"
+			(at 91.44 88.9 0)
+			(effects
+				(font
+					(size 1.27 1.27)
+				)
+				(hide yes)
+			)
+		)
+		(pin "3"
+		)
+		(pin "2"
+		)
+		(pin "1"
+		)
+		(pin "4"
+		)
+		(pin "5"
+		)
+		(pin "6"
+		)
+		(instances
+			(project "a1"
+				(path "/fc9f0664-12ec-44ef-b3db-0b33514ae060"
+					(reference "J1")
+					(unit 1)
+				)
+			)
+		)
+	)
+	(symbol
 		(lib_name "GND_6")
 		(lib_id "power:GND")
@@
 					(unit 1)
 				)
-			)
-		)
-	)
-	(symbol
-		(lib_id "Connector_Generic:Conn_02x03_Odd_Even")
-		(at 91.44 86.36 0)
-		(unit 1)
-		(exclude_from_sim no)
-		(in_bom yes)
-		(on_board yes)
-		(dnp no)
-		(property "Reference" "J1"
-			(at 92.71 80.772 0)
-			(effects
-				(font
-					(size 1.27 1.27)
-				)
-			)
-		)
-		(property "Value" "Conn_02x03_Odd_Even"
-			(at 93.218 73.406 0)
-			(effects
-				(font
-					(size 1.27 1.27)
-				)
-				(hide yes)
-			)
-		)
-		(property "Footprint" "Connector_PinHeader_2.54mm:PinHeader_2x03_P2.54mm_Vertical"
-			(at 91.44 86.36 0)
-			(effects
-				(font
-					(size 1.27 1.27)
-				)
-				(hide yes)
-			)
-		)
-		(property "Datasheet" "~"
-			(at 91.44 86.36 0)
-			(effects
-				(font
-					(size 1.27 1.27)
-				)
-				(hide yes)
-			)
-		)
-		(property "Description" "Generic connector, double row, 02x03, odd/even pin numbering scheme (row 1 odd numbers, row 2 even numbers), script generated (kicad-library-utils/schlib/autogen/connector/)"
-			(at 91.44 86.36 0)
-			(effects
-				(font
-					(size 1.27 1.27)
-				)
-				(hide yes)
-			)
-		)
-		(pin "3"
-		)
-		(pin "2"
-		)
-		(pin "1"
-		)
-		(pin "4"
-		)
-		(pin "5"
-		)
-		(pin "6"
-		)
-		(instances
-			(project "a0"
-				(path "/fc9f0664-12ec-44ef-b3db-0b33514ae060"
-					(reference "J1")
-					(unit 1)
-				)
